File: Nucleo_DAQ_Shield.sch (KiCad schematic (older format))
At the start: 32 parts, among them J1 CONN_01X06, J2 CONN_01X06, J3 CONN_01X02, J4 CONN_01X02, J6 CONN_COAXIAL, J7 CONN_01X02, U1 4050, U10 ST_Nucleo144_F746ZG_CN10, U2 TL072, U3 LM7805CT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

Commit message: Finalized v1.0 of PCB design
Connections:
- net VCC is gone; now on net +3.3VA: U1.1 (VCC), U1.1 (VCC), U1.1 (VCC)
- net VSS is gone; now on net GND: U1.8 (VSS), U1.8 (VSS), U1.8 (VSS)
Changed lines of the file:
@@
 Title "Nucleo DAQ Shield"
 Date "2017-07-11"
-Rev "v0.2"
+Rev "v1.0"
 Comp "Columbia University - Creative Machines Lab"
 Comment1 ""
@@
 $EndComp
 $Comp
-L +5V #PWR025
+L +5V #PWR023
 U 1 1 595D56EC
 P 800 1700
-F 0 "#PWR025" H 800 1550 50  0001 C CNN
+F 0 "#PWR023" H 800 1550 50  0001 C CNN
 F 1 "+5V" H 800 1840 50  0000 C CNN
 F 2 "" H 800 1700 50  0001 C CNN
@@
 $EndComp
 $Comp
-L +5VD #PWR026
+L +5VD #PWR024
 U 1 1 595D572D
 P 1000 1700
-F 0 "#PWR026" H 1000 1550 50  0001 C CNN
+F 0 "#PWR024" H 1000 1550 50  0001 C CNN
 F 1 "+5VD" H 1000 1840 50  0000 C CNN
 F 2 "" H 1000 1700 50  0001 C CNN
@@
 $EndComp
 $Comp
-L +5VA #PWR027
+L +5VA #PWR025
 U 1 1 595D5794
 P 1200 1700
-F 0 "#PWR027" H 1200 1550 50  0001 C CNN
+F 0 "#PWR025" H 1200 1550 50  0001 C CNN
 F 1 "+5VA" H 1200 1840 50  0000 C CNN
 F 2 "" H 1200 1700 50  0001 C CNN
@@
 $EndComp
 $Comp
-L +3.3VA #PWR028
+L +3.3VA #PWR026
 U 1 1 595D64A4
 P 1100 1400
-F 0 "#PWR028" H 1100 1250 50  0001 C CNN
+F 0 "#PWR026" H 1100 1250 50  0001 C CNN
 F 1 "+3.3VA" H 1100 1540 50  0000 C CNN
 F 2 "" H 1100 1400 50  0001 C CNN
@@
 $EndComp
 $Comp
-L +3.3V #PWR029
+L +3.3V #PWR027
 U 1 1 595D64EC
 P 800 1400
-F 0 "#PWR029" H 800 1250 50  0001 C CNN
+F 0 "#PWR027" H 800 1250 50  0001 C CNN
 F 1 "+3.3V" H 800 1540 50  0000 C CNN
 F 2 "" H 800 1400 50  0001 C CNN
@@
 $EndComp
 $Comp
-L GNDD #PWR030
+L GNDD #PWR028
 U 1 1 595E2075
 P 4450 3300
-F 0 "#PWR030" H 4450 3050 50  0001 C CNN
+F 0 "#PWR028" H 4450 3050 50  0001 C CNN
 F 1 "GNDD" H 4450 3150 50  0000 C CNN
 F 2 "" H 4450 3300 50  0001 C CNN
@@
 $EndComp
 $Comp
-L GNDD #PWR031
+L GNDD #PWR029
 U 1 1 595E228B
 P 5350 3450
-F 0 "#PWR031" H 5350 3200 50  0001 C CNN
+F 0 "#PWR029" H 5350 3200 50  0001 C CNN
 F 1 "GNDD" H 5350 3300 50  0000 C CNN
 F 2 "" H 5350 3450 50  0001 C CNN
@@
 $EndComp
 $Comp
-L GNDD #PWR032
+L GNDD #PWR030
 U 1 1 595E2DB5
 P 4250 4100
-F 0 "#PWR032" H 4250 3850 50  0001 C CNN
+F 0 "#PWR030" H 4250 3850 50  0001 C CNN
 F 1 "GNDD" H 4250 3950 50  0000 C CNN
 F 2 "" H 4250 4100 50  0001 C CNN
@@
 $EndComp
 $Comp
-L GNDD #PWR033
+L GNDD #PWR031
 U 1 1 595E3B16
 P 5500 3950
-F 0 "#PWR033" H 5500 3700 50  0001 C CNN
+F 0 "#PWR031" H 5500 3700 50  0001 C CNN
 F 1 "GNDD" H 5500 3800 50  0000 C CNN
 F 2 "" H 5500 3950 50  0001 C CNN
@@
 $EndComp
 $Comp
-L GNDD #PWR034
+L GNDD #PWR032
 U 1 1 595E3B7B
 P 5850 4300
-F 0 "#PWR034" H 5850 4050 50  0001 C CNN
+F 0 "#PWR032" H 5850 4050 50  0001 C CNN
 F 1 "GNDD" H 5850 4150 50  0000 C CNN
 F 2 "" H 5850 4300 50  0001 C CNN
@@
 ENCODER_X
 $Comp
-L GNDD #PWR035
+L GNDD #PWR033
 U 1 1 5964006B
 P 6600 1600
-F 0 "#PWR035" H 6600 1350 50  0001 C CNN
+F 0 "#PWR033" H 6600 1350 50  0001 C CNN
 F 1 "GNDD" H 6600 1450 50  0000 C CNN
 F 2 "" H 6600 1600 50  0001 C CNN
@@
 $EndComp
 $Comp
-L GNDD #PWR036
+L GNDD #PWR034
 U 1 1 59640685
 P 6700 3700
-F 0 "#PWR036" H 6700 3450 50  0001 C CNN
+F 0 "#PWR034" H 6700 3450 50  0001 C CNN
 F 1 "GNDD" H 6700 3550 50  0000 C CNN
 F 2 "" H 6700 3700 50  0001 C CNN
@@
 $EndComp
 $Comp
-L GNDD #PWR037
+L GNDD #PWR035
 U 1 1 596406F9
 P 7900 3100
-F 0 "#PWR037" H 7900 2850 50  0001 C CNN
+F 0 "#PWR035" H 7900 2850 50  0001 C CNN
 F 1 "GNDD" H 7900 2950 50  0000 C CNN
 F 2 "" H 7900 3100 50  0001 C CNN
@@
 $EndComp
 $Comp
-L GNDD #PWR038
+L GNDD #PWR036
 U 1 1 59640B64
 P 9000 3900
-F 0 "#PWR038" H 9000 3650 50  0001 C CNN
+F 0 "#PWR036" H 9000 3650 50  0001 C CNN
 F 1 "GNDD" H 9000 3750 50  0000 C CNN
 F 2 "" H 9000 3900 50  0001 C CNN
@@
 $EndComp
 $Comp
-L GNDD #PWR039
+L GNDD #PWR037
 U 1 1 59640BD8
 P 9000 3400
-F 0 "#PWR039" H 9000 3150 50  0001 C CNN
+F 0 "#PWR037" H 9000 3150 50  0001 C CNN
 F 1 "GNDD" H 9000 3250 50  0000 C CNN
 F 2 "" H 9000 3400 50  0001 C CNN
@@
 $EndComp
 $Comp
-L GNDD #PWR040
+L GNDD #PWR038
 U 1 1 59640C4C
 P 10200 3600
-F 0 "#PWR040" H 10200 3350 50  0001 C CNN
+F 0 "#PWR038" H 10200 3350 50  0001 C CNN
 F 1 "GNDD" H 10200 3450 50  0000 C CNN
 F 2 "" H 10200 3600 50  0001 C CNN
@@
 $EndComp
 $Comp
-L GNDD #PWR041
+L GNDD #PWR039
 U 1 1 59640CC0
 P 9000 2800
-F 0 "#PWR041" H 9000 2550 50  0001 C CNN
+F 0 "#PWR039" H 9000 2550 50  0001 C CNN
 F 1 "GNDD" H 9000 2650 50  0000 C CNN
 F 2 "" H 9000 2800 50  0001 C CNN
@@
 $EndComp
 $Comp
-L GNDD #PWR042
+L GNDD #PWR040
 U 1 1 59641036
 P 10050 1400
-F 0 "#PWR042" H 10050 1150 50  0001 C CNN
+F 0 "#PWR040" H 10050 1150 50  0001 C CNN
 F 1 "GNDD" H 10050 1250 50  0000 C CNN
 F 2 "" H 10050 1400 50  0001 C CNN
@@
 $EndComp
 $Comp
-L GNDA #PWR043
+L GNDA #PWR041
 U 1 1 596414C2
 P 8800 2700
-F 0 "#PWR043" H 8800 2450 50  0001 C CNN
+F 0 "#PWR041" H 8800 2450 50  0001 C CNN
 F 1 "GNDA" H 8800 2550 50  0000 C CNN
 F 2 "" H 8800 2700 50  0001 C CNN
@@
 $EndComp
 $Comp
-L GNDD #PWR044
+L GNDD #PWR042
 U 1 1 59640585
 P 3700 7100
-F 0 "#PWR044" H 3700 6850 50  0001 C CNN
+F 0 "#PWR042" H 3700 6850 50  0001 C CNN
 F 1 "GNDD" H 3700 6950 50  0000 C CNN
 F 2 "" H 3700 7100 50  0001 C CNN
@@
 $EndComp
 $Comp
-L +3.3V #PWR045
+L +3.3V #PWR043
 U 1 1 596405FC
 P 3700 6900
-F 0 "#PWR045" H 3700 6750 50  0001 C CNN
+F 0 "#PWR043" H 3700 6750 50  0001 C CNN
 F 1 "+3.3V" H 3700 7040 50  0000 C CNN
 F 2 "" H 3700 6900 50  0001 C CNN
@@
 $EndComp
 $Comp
-L GNDD #PWR046
+L GNDD #PWR044
 U 1 1 596410E3
 P 4100 7100
-F 0 "#PWR046" H 4100 6850 50  0001 C CNN
+F 0 "#PWR044" H 4100 6850 50  0001 C CNN
 F 1 "GNDD" H 4100 6950 50  0000 C CNN
 F 2 "" H 4100 7100 50  0001 C CNN
@@
 $EndComp
 $Comp
-L +3.3V #PWR047
+L +3.3V #PWR045
 U 1 1 596410E9
 P 4100 6900
-F 0 "#PWR047" H 4100 6750 50  0001 C CNN
+F 0 "#PWR045" H 4100 6750 50  0001 C CNN
 F 1 "+3.3V" H 4100 7040 50  0000 C CNN
 F 2 "" H 4100 6900 50  0001 C CNN
@@
 $EndComp
 $Comp
-L GNDD #PWR048
+L GNDD #PWR046
 U 1 1 596424FC
 P 2100 5800
-F 0 "#PWR048" H 2100 5550 50  0001 C CNN
+F 0 "#PWR046" H 2100 5550 50  0001 C CNN
 F 1 "GNDD" H 2100 5650 50  0000 C CNN
 F 2 "" H 2100 5800 50  0001 C CNN
@@
 $EndComp
 $Comp
-L GNDD #PWR049
+L GNDD #PWR047
 U 1 1 5965067E
 P 1200 5900
-F 0 "#PWR049" H 1200 5650 50  0001 C CNN
+F 0 "#PWR047" H 1200 5650 50  0001 C CNN
 F 1 "GNDD" H 1200 5750 50  0000 C CNN
 F 2 "" H 1200 5900 50  0001 C CNN
@@
 $EndComp
 $Comp
-L GNDA #PWR050
+L GNDA #PWR048
 U 1 1 5965449B
 P 5600 6100
-F 0 "#PWR050" H 5600 5850 50  0001 C CNN
+F 0 "#PWR048" H 5600 5850 50  0001 C CNN
 F 1 "GNDA" H 5600 5950 50  0000 C CNN
 F 2 "" H 5600 6100 50  0001 C CNN
@@
 $EndComp
 $Comp
-L GNDA #PWR051
+L GNDA #PWR049
 U 1 1 59654512
 P 5400 6100
-F 0 "#PWR051" H 5400 5850 50  0001 C CNN
+F 0 "#PWR049" H 5400 5850 50  0001 C CNN
 F 1 "GNDA" H 5400 5950 50  0000 C CNN
 F 2 "" H 5400 6100 50  0001 C CNN
@@
 Text Notes 5000 5700 0    30   ~ 0
 SMA connector
+$Comp
+L +3.3V #PWR050
+U 1 1 59658F3C
+P 2100 4300
+F 0 "#PWR050" H 2100 4150 50  0001 C CNN
+F 1 "+3.3V" H 2100 4440 50  0000 C CNN
+F 2 "" H 2100 4300 50  0001 C CNN
+F 3 "" H 2100 4300 50  0001 C CNN
+	1    2100 4300
+	1    0    0    -1
+$EndComp
+$Comp
+L GNDD #PWR051
+U 1 1 59659154
+P 2100 4900
+F 0 "#PWR051" H 2100 4650 50  0001 C CNN
+F 1 "GNDD" H 2100 4750 50  0000 C CNN
+F 2 "" H 2100 4900 50  0001 C CNN
+F 3 "" H 2100 4900 50  0001 C CNN
+	1    2100 4900
+	1    0    0    -1
+$EndComp
+Wire Wire Line
+	2100 4700 1900 4700
+Wire Wire Line
+	1900 4700 1900 4650
+$Comp
+L +3.3V #PWR052
+U 1 1 5965984E
+P 1900 4650
+F 0 "#PWR052" H 1900 4500 50  0001 C CNN
+F 1 "+3.3V" H 1900 4790 50  0000 C CNN
+F 2 "" H 1900 4650 50  0001 C CNN
+F 3 "" H 1900 4650 50  0001 C CNN
+	1    1900 4650
+	1    0    0    -1
+$EndComp
+$Comp
+L GNDD #PWR053
+U 1 1 596598C2
+P 2100 4500
+F 0 "#PWR053" H 2100 4250 50  0001 C CNN
+F 1 "GNDD" H 2100 4350 50  0000 C CNN
+F 2 "" H 2100 4500 50  0001 C CNN
+F 3 "" H 2100 4500 50  0001 C CNN
+	1    2100 4500
+	1    0    0    -1
+$EndComp
+$Comp
+L GNDD #PWR054
+U 1 1 59659C32
+P 1600 5800
+F 0 "#PWR054" H 1600 5550 50  0001 C CNN
+F 1 "GNDD" H 1600 5650 50  0000 C CNN
+F 2 "" H 1600 5800 50  0001 C CNN
+F 3 "" H 1600 5800 50  0001 C CNN
+	1    1600 5800
+	1    0    0    -1
+$EndComp
+$Comp
+L +3.3V #PWR055
+U 1 1 59659DBE
+P 1600 5600
+F 0 "#PWR055" H 1600 5450 50  0001 C CNN
+F 1 "+3.3V" H 1600 5740 50  0000 C CNN
+F 2 "" H 1600 5600 50  0001 C CNN
+F 3 "" H 1600 5600 50  0001 C CNN
+	1    1600 5600
+	1    0    0    -1
+$EndComp
 $EndSCHEMATC
